Commit message: pan_tilt implementation with xacro

File: urdf/pan_tilt.xacro (robot description, xacro)
@@ -1,4 +1,21 @@
 <?xml version="1.0"?>
-<robot name="pan_tilt"><!-- Its elements are <link>,<joint>,<transmission>,<gazebo>-->
+<robot
+    xmlns:xacro="http://www.ros.org/wiki/xacro"
+    xmlns:sensor="htttp:/playerstage.sourceforce.net/gazebo/xmlschema/#sensor"
+    xmlns:controller="htttp:/playerstage.sourceforce.net/gazebo/xmlschema/#controller"
+    xmlns:interface="htttp:/playerstage.sourceforce.net/gazebo/xmlschema/#interface"
+    name="pan_tilt" >
+    <xacro:property name="base_link_length" value="0.05"  />
+    <xacro:property name="base_link_radius" value="0.2"  />
+    <xacro:property name="pan_link_length" value="0.5"  />
+    <xacro:property name="pan_link_radius" value="0.02"  />
+    <xacro:property name="bearing_radius" value="0.02"  />
+    <xacro:property name="tilt_link_size" value="0.5 0.5 0.03"  />
+    <xacro:macro name="inertial_matrix" params="mass">
+        <inertial>
+            <mass value="${mass}"/>
+            <inertia ixx="1" ixy="0" ixz="0" iyy="1" iyz="0" izz="1" />
+        </inertial>
+    </xacro:macro>
     <material name="yellow">
         <color rgba="1 1 0 1" />
@@ -16,5 +33,5 @@
         <visual>
             <geometry>
-                <cylinder length="0.05" radius="0.2"/>
+                <cylinder length="${base_link_length}" radius="${base_link_radius}"/>
             </geometry>
             <origin xyz="0 0 0.025" rpy="0 0 0 " />
@@ -23,22 +40,15 @@
         <collision>
             <geometry>
-                <cylinder length="0.055" radius="0.25"/>
+                <cylinder length="${base_link_length+0.05}" radius="${base_link_radius+0.05}"/>
             </geometry>
             <origin xyz="0 0 0.025" rpy="0 0 0 " />
         </collision>
-        <!--[ WARN] [1656079412.718004450]:
-            The root link base_link has an inertia specified in the URDF,
-            but KDL does not support a root link with an inertia.
-            As a workaround, you can add an extra dummy link to your URDF.
-        <inertial>
-            <origin xyz="0 0 0 " rpy="0 0 0 " />
-            <mass value="1" />
-            <inertia ixx="1" ixy="0" ixz="0" iyy="1" iyz="0" izz="1" />
-        </inertial>  -->
+        <!-- KDL does not support a root link with an inertia.
+            As a workaround, you can add an extra dummy link to your URDF. -->
     </link>
     <link name="pan_link">
         <visual>
             <geometry>
-                <cylinder length="0.5" radius="0.02" />
+                <cylinder length="${pan_link_length}" radius="${pan_link_radius}" />
             </geometry>
             <origin xyz="0 0 0.25" rpy="0 0 0 " />
@@ -47,13 +57,9 @@
         <collision>
             <geometry>
-                <cylinder length="0.55" radius="0.025"/>
+                <cylinder length="${pan_link_length+0.05}" radius="${pan_link_radius+0.05}" />
             </geometry>
             <origin xyz="0 0 0.25" rpy="0 0 0 " />
         </collision>
-        <inertial>
-            <origin xyz="0 0 0.25 " rpy="0 0 0 " />
-            <mass value="1" />
-            <inertia ixx="1" ixy="0" ixz="0" iyy="1" iyz="0" izz="1" />
-        </inertial>
+        <xacro:inertial_matrix mass="1" />
     </link>
     <joint name="pan_joint"  type="revolute">
@@ -69,5 +75,5 @@
             <origin xyz="0 0 0" rpy="0 0 0 " />
             <geometry>
-                <sphere radius="0.02" />
+                <sphere radius="${bearing_radius}" />
             </geometry>
             <material name="white" />
@@ -76,12 +82,8 @@
             <origin xyz="0 0 0" rpy="0 0 0 " />
             <geometry>
-                <sphere radius="0.11" />
+                <sphere radius="${bearing_radius+0.05}" />
             </geometry>
         </collision>
-        <inertial>
-            <origin xyz="0 0 0" rpy="0 0 0 " />
-            <mass value="1" />
-            <inertia ixx="1" ixy="0" ixz="0" iyy="1" iyz="0" izz="1" />
-        </inertial>
+        <xacro:inertial_matrix mass="1" />
     </link>
     <joint name="bearing_joint" type="fixed">
@@ -94,5 +96,5 @@
             <origin xyz="0 0 0" rpy="0 0 0 " />
             <geometry>
-                <box size="0.5 0.5 0.03" />
+                <box size="${tilt_link_size}" />
             </geometry>
             <material name="green" />
@@ -101,12 +103,8 @@
             <origin xyz="0 0 0" rpy="0 0 0 " />
             <geometry>
-                <box size="0.11 0.11 0.031" />
+                <box size="0.55 0.55 0.035" />
             </geometry>
         </collision>
-        <inertial>
-            <origin xyz="0 0 0" rpy="0 0 0 " />
-            <mass value="1" />
-            <inertia ixx="1" ixy="0" ixz="0" iyy="1" iyz="0" izz="1" />
-        </inertial>
+        <xacro:inertial_matrix mass="1" />
     </link>
     <joint name="tilt_joint" type="revolute">
